File: rs_485_proje.kicad_sch (KiCad schematic)
At the start: 54 parts, among them J2 RJ45_LED, J3 Piezzo_2, J4 Led_conn, J5 Piezzo_1, J6 USB_B_Mini, J7 H_E_sensor_1, J8 H_E_sensor_2, J9 Debug, U1 AP2112K-3.3, U10 FT232RL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

Commit message: 12.04.2026/11:46
Parts:
- removed C16, C17: 100nf, Capacitor_SMD:C_0805_2012Metric, symbol Device:C
- removed D2: SM712_SOT23, Package_TO_SOT_SMD:SOT-23, symbol Diode:SM712_SOT23
- removed R15, R16: 10K, Resistor_SMD:R_0805_2012Metric, symbol Device:R_US
- removed U3: SN65HVD1781, Package_SO:SOIC-8_3.9x4.9mm_P1.27mm, symbol Interface_UART:SN65HVD1781
- removed U6: ISO7241CDWR, Package_SO:SOIC-16W-12_7.5x10.3mm_P1.27mm, symbol isalatör:ISO7241CDWR
- added C13, C14: 100nF, Capacitor_SMD:C_0805_2012Metric, symbol Device:C
- added D6: SM712_SOT23, Package_TO_SOT_SMD:SOT-23, symbol Diode:SM712_SOT23
- added R17, R18: 10K, Resistor_SMD:R_0805_2012Metric, symbol Device:R_US
- added R19: 120R, Resistor_SMD:R_0805_2012Metric, symbol Device:R_US
- C11, C12, C3, C4, C6: value 100nf -> 100nF
- R3: value 120R -> 10K
Connections:
- net +3.3V_USB is gone; now on net +3.3V: U10.4 (VCCIO)
- net +5V_USB is gone; now on net +5V: C15.1, U10.20 (VCC)
- net USB_GND is gone; now on net GND: C15.2, J6.5 (GND), U10.18 (GND), U10.21 (GND), U10.7 (GND), U11.2 (GND)
- net +24V: now also R3.1
- net +3.3V: now also C12.1, C6.2; no longer C11.1, C6.1
- net GND: now also C12.2, C6.1, J6.SH (Shield), U10.25 (AGND), U10.26 (TEST), U4.1 (GND1), U4.10 (GND1), U4.3 (GND1), U4.9 (GND1), C13.2, C14.2; no longer C11.2, C6.2
- net GNDB: now also C11.2, U4.11 (GND2), U4.14 (GND2), D6.3 (common); no longer C12.2
- net RS485_A(-): now also U4.13 (Y), U4.18 (A), D6.1 (A1), R19.1; no longer R3.1
- net RS485_B(+): now also U4.15 (Z), U4.17 (B), D6.2 (A2), R19.2; no longer R3.2
- net RS_485_D_EN: now also U4.6 (DE)
- net RS_485_R_EN: now also U4.5 (~{RE})
- net UART_1_RX: now also U4.4 (RxD)
- net UART_1_TX: now also U4.7 (TxD)
- net at D1.1 (K), L1.1, U5.8 (PH): now also C3.2; no longer C3.1
- net at U5.1 (BOOT): now also C3.1; no longer C3.2
- net at U5.5 (ENA): now also R3.2
- net +3V3: now reaches U4.12 (Visoout)
- net +3V3: now also C11.1, C4.1, U4.19 (Visoin), R17.2, R18.2
- net at U4.16 (GND2): now also U4.20 (GND2)
- net at U4.2 (VCC): now also R18.1
- net at U4.8 (VCC): now also R17.1
- net at D5.2 (A), J6.1 (VBUS), U11.5 (VBUS): now also C13.1
- net at U10.17 (3V3OUT): now also C14.1
- removed net +3V3B: C12.1, C4.1
- no-connect marks 3 -> 18
Other:
- note added: "+5V"
- note added: "3.3V"
- note added: "HALL EFFECT SENSOR"
- note added: "PIEZZO SENSOR"
- note added: "POWER"
- note added: "RS485"
- moved on the sheet: U4

Commit message: 12.04.2026\15.40
Parts:
- removed R17, R18: 10K, Resistor_SMD:R_0805_2012Metric, symbol Device:R_US
- added C16, C17: 100nF, Capacitor_SMD:C_0805_2012Metric, symbol Device:C
Connections:
- net +3V3: now also U4.2 (VCC), U4.8 (VCC), C16.2, C17.2
- net GND: now also C16.1, C17.1
- net GNDB: now also U4.16 (GND2), U4.20 (GND2)

Commit message: 26.04.2026/10:37
Parts:
- added C18: 4.7uf, Capacitor_THT:C_Radial_D5.0mm_H11.0mm_P2.00mm, symbol Device:C_US
- added C19, C20: 4.7nf, Capacitor_SMD:C_0805_2012Metric, symbol Device:C
- added D10, D12, D13, D9: D_Schottky, symbol Device:D_Schottky
- added D11, D14: 3.3V, Diode_SMD:D_SOD-123, symbol Device:D_Zener
- added D2, D7, D8: LED, symbol Device:LED
- added J1: Piezzo_1, symbol Connector_Generic:Conn_01x02
- added J10: Piezzo_2, symbol Connector_Generic:Conn_01x02
- added R15, R16: 2.3K, Resistor_SMD:R_0805_2012Metric, symbol Device:R_US
- added R17, R18: 1M, Resistor_SMD:R_0805_2012Metric, symbol Device:R_US
- C1: value 10uf -> 4.7uf
- C9: value 4.5n -> 4.7nf
Connections:
- net +24V: now also C18.1
- net +3.3V: now also R15.2, R16.2
- net +3V3: no longer C11.1, C4.1, U4.12 (Visoout), U4.19 (Visoin)
- net GND: now also C18.2, C19.1, C20.1, D10.2 (A), D11.2 (A), D13.2 (A), D14.2 (A), J1.2 (Pin_2), J10.2 (Pin_2), R17.2, R18.2
- net Piezzo_sens_1: now also C19.2, D10.1 (K), D11.1 (K), D9.1 (K), J1.1 (Pin_1), R17.1
- net Piezzo_sens_2: now also C20.2, D12.1 (K), D13.1 (K), D14.1 (K), J10.1 (Pin_1), R18.1
- net UART_2_RX: now also D8.1 (K)
- net UART_2_TX: now also D2.1 (K)
- new net: D2.2 (A), R15.1
- new net: D8.2 (A), R16.1
- new net +3V3B: C11.1, C4.1, U4.12 (Visoout), U4.19 (Visoin)
Other:
- moved on the sheet: C1, C10, C9, D3, D4, J3, J5, R1, R2, R3, R6, R8

Commit message: 26/04/12:18
Parts:
- removed D10, D12, D13, D9: D_Schottky, symbol Device:D_Schottky
- removed D11, D14: 3.3V, Diode_SMD:D_SOD-123, symbol Device:D_Zener
- added D10, D12, D15, D9: 1N5819, Diode_THT:D_DO-41_SOD81_P10.16mm_Horizontal, symbol Diode:1N5819
- added D11, D13: BZX84Cxx, Package_TO_SOT_SMD:SOT-23, symbol Diode:BZX84Cxx
- added J11, J12: P_E_sensor_1, symbol Connector_Generic:Conn_01x03
- added R20: 330R, Resistor_SMD:R_0805_2012Metric, symbol Device:R_US
- added R21: 10K, Resistor_SMD:R_0805_2012Metric, symbol Device:R_US
- R15, R16: value 2.3K -> 330R
Connections:
- net GND: now also D10.2 (A), D11.1 (A), D13.1 (A), D9.2 (A), J11.1 (Pin_1), J12.1 (Pin_1), R21.2
- net LED_Driver: now also R20.1; no longer J4.2 (Pin_2)
- net Piezzo_sens_1: now also D10.1 (K), D12.1 (K), D13.3 (K)
- net Piezzo_sens_2: now also D11.3 (K), D15.1 (K), D9.1 (K)
- net UART_2_RX: no longer D8.1 (K)
- net UART_2_TX: no longer D2.1 (K)
- net at U10.22 (CBUS1): now also D2.1 (K)
- net at U10.23 (CBUS0): now also D8.1 (K)
- new net: D15.2 (A), J12.3 (Pin_3)
- new net: D12.2 (A), J11.3 (Pin_3)
- new net: J4.2 (Pin_2), R20.2, R21.1
- no-connect marks 18 -> 16
Other:
- moved on the sheet: C20, D2, D8, J10, J4, R15, R16, R18

Commit message: 26/04/12:32
Parts:
- removed R3: 10K, Resistor_SMD:R_0805_2012Metric, symbol Device:R_US
Connections:
- no-connect marks 16 -> 17
Changed lines of the file:
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@@
 	)
 	(junction
-		(at 30.48 154.94)
-		(diameter 0)
-		(color 0 0 0 0)
-	)
-	(junction
 		(at 76.2 151.13)
 		(diameter 0)
@@
 	)
 	(no_connect
+		(at 34.29 160.02)
+	)
+	(no_connect
 		(at 346.71 179.07)
 	)
@@
 		)
 	)
-	(wire
-		(pts
-			(xy 30.48 166.37) (xy 34.29 166.37)
-		)
-		(stroke
-			(width 0)
-			(type default)
-		)
-	)
 	(polyline
 		(pts
@@
 	(wire
 		(pts
-			(xy 24.13 154.94) (xy 30.48 154.94)
-		)
-		(stroke
-			(width 0)
-			(type default)
-		)
-	)
-	(wire
-		(pts
 			(xy 349.25 162.56) (xy 349.25 161.29)
 		)
@@
 	(wire
 		(pts
-			(xy 30.48 154.94) (xy 34.29 154.94)
+			(xy 24.13 154.94) (xy 34.29 154.94)
 		)
 		(stroke
@@
 	(wire
 		(pts
-			(xy 34.29 166.37) (xy 34.29 160.02)
-		)
-		(stroke
-			(width 0)
-			(type default)
-		)
-	)
-	(wire
-		(pts
 			(xy 15.24 52.07) (xy 29.21 52.07)
 		)
@@
 	(wire
 		(pts
-			(xy 30.48 154.94) (xy 30.48 156.21)
-		)
-		(stroke
-			(width 0)
-			(type default)
-		)
-	)
-	(wire
-		(pts
 			(xy 35.56 228.6) (xy 44.45 228.6)
 		)
@@
 	(wire
 		(pts
-			(xy 30.48 163.83) (xy 30.48 166.37)
-		)
-		(stroke
-			(width 0)
-			(type default)
-		)
-	)
-	(wire
-		(pts
 			(xy 26.67 251.46) (xy 33.02 251.46)
 		)
@@
 					(unit 1)
 				)
-			)
-		)
-	)
-	(symbol
-		(lib_id "Device:R_US")
-		(at 30.48 160.02 0)
-		(unit 1)
-		(exclude_from_sim no)
-		(in_bom yes)
-		(on_board yes)
-		(dnp no)
-		(property "Reference" "R3"
-			(at 32.512 164.338 0)
-			(effects
-				(font
-					(size 1.27 1.27)
-				)
-			)
-		)
-		(property "Value" "10K"
-			(at 32.512 166.116 0)
-			(effects
-				(font
-					(size 1.27 1.27)
-				)
-			)
-		)
-		(property "Footprint" "Resistor_SMD:R_0805_2012Metric"
-			(at 31.496 160.274 90)
-			(effects
-				(font
-					(size 1.27 1.27)
-				)
-				(hide yes)
-			)
-		)
-		(property "Datasheet" ""
-			(at 30.48 160.02 0)
-			(effects
-				(font
-					(size 1.27 1.27)
-				)
-				(hide yes)
-			)
-		)
-		(property "Description" "Resistor, US symbol"
-			(at 30.48 160.02 0)
-			(effects
-				(font
-					(size 1.27 1.27)
-				)
-				(hide yes)
-			)
-		)
-		(pin "2"
-		)
-		(pin "1"
-		)
-		(instances
-			(project "rs_485_proje"
-				(path "/c9918559-5512-44e8-b15e-1805e85a5c10"
-					(reference "R3")
-					(unit 1)
-				)

Commit message: 26/04/14:43
Parts:
- removed C10: 4.5n, Capacitor_SMD:C_0805_2012Metric, symbol Device:C
- removed C9: 4.7nf, Capacitor_SMD:C_0805_2012Metric, symbol Device:C
- removed D3, D4: 3.3V, Diode_SMD:D_SOD-123, symbol Device:D_Zener
- removed D7: LED, symbol Device:LED
- removed J11, J12: P_E_sensor_1, symbol Connector_Generic:Conn_01x03
- removed J3: Piezzo_2, symbol Connector_Generic:Conn_01x02
- removed J5: Piezzo_1, symbol Connector_Generic:Conn_01x02
- removed R1, R2, R6, R8: 1M, Resistor_SMD:R_0805_2012Metric, symbol Device:R_US
- added J11: P_E_SENSOR_1, symbol Connector_Generic:Conn_01x02
- added J12: P_E_SENSOR_2, symbol Connector_Generic:Conn_01x02
Connections:
- net Digital_sens_1: no longer U2.11 (PA4)
- net Digital_sens_2: no longer U2.12 (PA5)
- net GND: now also J11.1 (Pin_1), J12.1 (Pin_1)
- net SENS_3: now also U2.11 (PA4)
- net SENS_4: now also U2.12 (PA5)
- net at D15.2 (A): now also J12.2 (Pin_2)
- net at D12.2 (A): now also J11.2 (Pin_2)

Commit message: 26/04/18:51
Parts:
- removed J1: Piezzo_1, symbol Connector_Generic:Conn_01x02
- removed J10: Piezzo_2, symbol Connector_Generic:Conn_01x02

Commit message: 27/04/15:17
Parts:
- removed D5: D_Schottky, symbol Device:D_Schottky
- added D3, D4, D5: 1N5819, Diode_THT:D_DO-41_SOD81_P10.16mm_Horizontal, symbol Diode:1N5819
- added J1: xt60_female, Connector_AMASS:AMASS_XT60-F_1x02_P7.20mm_Vertical, symbol Connector_Generic:Conn_01x02
Connections:
- net +24V: now also D4.1 (K)
- net +5V: now also D3.1 (K)
- net GND: now also D5.1 (K)
- net at C13.1, J6.1 (VBUS), U11.5 (VBUS): now also D3.2 (A)
- new net: D4.2 (A), J1.1 (Pin_1)
- new net: D5.2 (A), J1.2 (Pin_2)
Other:
- moved on the sheet: R20, R21
