File: rs_485_proje.kicad_sch (KiCad schematic)
At the start: 64 parts, among them J1 xt60_female, J11 P_E_SENSOR_1, J12 P_E_SENSOR_2, J2 RJ45_LED, J4 Led_conn, J6 USB_B_Mini, J7 H_E_sensor_1, J8 H_E_sensor_2, J9 Debug, U1 AP2112K-3.3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

Commit message: Şematik neredeyse son haline getirildi. Bazı kozmetik düzeltmeler yapıldı.
Parts:
- removed C19: 4.7nf, Capacitor_SMD:C_0805_2012Metric, symbol Device:C
- removed D10, D12: 1N5819, Diode_THT:D_DO-41_SOD81_P10.16mm_Horizontal, symbol Diode:1N5819
- removed D13: BZX84Cxx, Package_TO_SOT_SMD:SOT-23, symbol Diode:BZX84Cxx
- removed J11: P_E_SENSOR_1, symbol Connector_Generic:Conn_01x02
- removed R17: 1M, Resistor_SMD:R_0805_2012Metric, symbol Device:R_US
- added C9: 4.7nf, Capacitor_SMD:C_0805_2012Metric, symbol Device:C
- added D14: BZX84Cxx, Package_TO_SOT_SMD:SOT-23, symbol Diode:BZX84Cxx
- added D7: 1N5819, Diode_THT:D_DO-41_SOD81_P10.16mm_Horizontal, symbol Diode:1N5819
- added J10: Extra_pins, symbol Connector:Conn_01x06_Pin
- added J3: xt60_female, Connector_AMASS:AMASS_XT60-F_1x02_P7.20mm_Vertical, symbol Connector_Generic:Conn_01x02
- added J5: P_E_SENSOR_1, symbol Connector_Generic:Conn_01x02
- added R1: 1M, Resistor_SMD:R_0805_2012Metric, symbol Device:R_US
Connections:
- net SENS_3 is gone; now on net Digital_sens_1: R13.1, U2.11 (PA4), U7.7 (VO1)
- net SENS_4 is gone; now on net Digital_sens_2: R14.1, U2.12 (PA5), U7.6 (VO2)
- net +24V: now also J10.2 (Pin_2)
- net +3.3V: now also J10.4 (Pin_4)
- net +5V: now also J10.3 (Pin_3)
- net Digital_sens_1: no longer J7.2 (Pin_2), R11.2, U7.1 (A1)
- net Digital_sens_2: no longer J8.2 (Pin_2), R12.2, U7.3 (C2)
- net GND: now also J1.2 (Pin_2), C9.1, D14.1 (A), D7.2 (A), J10.1 (Pin_1), J3.2 (Pin_2), J5.1 (Pin_1), R1.2; no longer D5.1 (K)
- net Piezzo_sens_1: now also D5.1 (K), C9.2, D14.3 (K), D7.1 (K), R1.1
- net at D4.2 (A), J1.1 (Pin_1): now also J3.1 (Pin_1)
- net at D5.2 (A): now also J5.2 (Pin_2); no longer J1.2 (Pin_2)
- net Extra_1 renamed PA_6
- net PA_6: now also J10.6 (Pin_6); no longer U2.14 (PA7)
- new net PA_7: J10.5 (Pin_5), U2.14 (PA7)
- new net d_sens_1: J7.2 (Pin_2), R11.2, U7.1 (A1)
- new net d_sens_2: J8.2 (Pin_2), R12.2, U7.3 (C2)
Other:
- note added: "External 24V"
- note added: "Extra"
- note added: "RGB Addressed Led"
- note added: "UART-USB"
- note removed: "NOT: Bu 24V ayrı olmalı. çünkü bu harici bağlanacak"
- note removed: "NOT: Ena boşta kalmış. Kapasiteler doğru mu?"
- note removed: "NOT: LEd driver'e buffer veya optocoupler koyulaiblir"
- note removed: "NOT: Pin yapısını kontrol et."
- note removed: "NOT: Yeni RS-485 entegresi eklenecek"
- moved on the sheet: C1, C11, C12, C13, C14, C15, C16, C17, C18, C2, C20, C3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

Commit message: -Şematikte bazı değişimler yapılıd. -İzole Rs-485 entegresine ek kapasitörler eklendi. -Addreslenebilir lede giden 24V'nin sadece harici pil takılıdğında çalışması sağlandı.
Parts:
- removed C11, C16, C17, C4: 100nF, Capacitor_SMD:C_0805_2012Metric, symbol Device:C
- removed C9: 4.7nf, Capacitor_SMD:C_0805_2012Metric, symbol Device:C
- removed R1: 1M, Resistor_SMD:R_0805_2012Metric, symbol Device:R_US
- added C10, C11, C16, C4: 100nf, symbol Device:C_Small
- added C17: 4.7f, symbol Device:C_Small
- added C19, C21: 10uf, symbol Device:C_Polarized_Small
- added C22, C9: 10nf, symbol Device:C_Small
- added R2: 1M, symbol Device:R_Small
Connections:
- net +24V: no longer J4.3 (Pin_3)
- net +3V3B: now also C10.1, C19.1, C4.1, C9.1
- net +5V: no longer C2.1, C7.2, J10.3 (Pin_3), L1.2, R12.1, R4.1, U1.1 (VIN), U1.3 (EN)
- net GND: now also U7.3 (C2), C11.1, C16.1, C17.2, C21.1, C22.1, R2.2; no longer U7.4 (A2)
- net GNDB: now also C10.2, C19.2, C4.2, C9.2
- net Piezzo_sens_1: now also C17.1, R2.1
- net +3V3: no longer names the net of U4.2 (VCC), U4.8 (VCC)
- net +3V3: now also C11.2, C16.2, C21.2, C22.2
- net d_sens_1: no longer names the net of J7.2 (Pin_2), R11.2, U7.1 (A1)
- net d_sens_2: no longer names the net of J8.2 (Pin_2), R12.2
- net d_sens_2: now also U7.4 (A2); no longer U7.3 (C2)
- new net: C2.1, L1.2
- new net: C7.2, U1.1 (VIN), U1.3 (EN)
Other:
- note added: "NOT: -Görseldeki kurallara uyulmalı. -Tüm pinler için power input output ayarlanmalı."
- moved on the sheet: J8, R11, R12

Commit message: 11/05/2026/11:52
Parts:
- J10: footprint (none) -> Connector_PinHeader_2.54mm:PinHeader_1x06_P2.54mm_Vertical
- J12, J5: footprint (none) -> TerminalBlock_Phoenix:TerminalBlock_Phoenix_PT-1,5-2-3.5-H_1x02_P3.50mm_Horizontal
- J4: footprint (none) -> Connector_PinHeader_2.54mm:PinHeader_1x03_P2.54mm_Vertical
- J7, J8: footprint (none) -> TerminalBlock_Phoenix:TerminalBlock_Phoenix_PT-1,5-3-3.5-H_1x03_P3.50mm_Horizontal
- J9: footprint (none) -> Connector_PinHeader_2.54mm:PinHeader_1x04_P2.54mm_Vertical
Changed lines of the file:
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@@
 			)
 		)
-		(property "Footprint" ""
+		(property "Footprint" "TerminalBlock_Phoenix:TerminalBlock_Phoenix_PT-1,5-3-3.5-H_1x03_P3.50mm_Horizontal"
 			(at 111.76 30.48 0)
 			(effects
@@
 			)
 		)
-		(property "Footprint" ""
+		(property "Footprint" "Connector_PinHeader_2.54mm:PinHeader_1x04_P2.54mm_Vertical"
 			(at 86.36 22.86 0)
 			(effects
@@
 			)
 		)
-		(property "Footprint" ""
+		(property "Footprint" "TerminalBlock_Phoenix:TerminalBlock_Phoenix_PT-1,5-2-3.5-H_1x02_P3.50mm_Horizontal"
 			(at 129.54 104.14 0)
 			(effects
@@
 			)
 		)
-		(property "Footprint" ""
+		(property "Footprint" "TerminalBlock_Phoenix:TerminalBlock_Phoenix_PT-1,5-2-3.5-H_1x02_P3.50mm_Horizontal"
 			(at 129.54 73.66 0)
 			(effects
@@
 			)
 		)
-		(property "Footprint" ""
+		(property "Footprint" "TerminalBlock_Phoenix:TerminalBlock_Phoenix_PT-1,5-3-3.5-H_1x03_P3.50mm_Horizontal"
 			(at 111.76 46.99 0)
 			(effects
@@
 			)
 		)
-		(property "Footprint" ""
+		(property "Footprint" "Connector_PinHeader_2.54mm:PinHeader_1x06_P2.54mm_Vertical"
 			(at 168.91 208.28 0)
 			(effects
@@
 			)
 		)
-		(property "Footprint" ""
+		(property "Footprint" "Connector_PinHeader_2.54mm:PinHeader_1x03_P2.54mm_Vertical"
 			(at 62.23 256.54 0)
 			(effects

Commit message: 11/05/16:16
Parts:
- removed C10, C11, C16, C4, C5: 100nf, symbol Device:C_Small
- removed C17: 4.7f, symbol Device:C_Small
- removed R2: 1M, symbol Device:R_Small
- added C10, C11, C16, C4, C5: 100nF, Capacitor_SMD:C_0805_2012Metric, symbol Device:C
- added C17: 4.7nf, Capacitor_SMD:C_0805_2012Metric, symbol Device:C
- added R1: 1M, Resistor_SMD:R_0805_2012Metric, symbol Device:R_US
- C1, C18: footprint Capacitor_THT:C_Radial_D5.0mm_H11.0mm_P2.00mm -> Capacitor_SMD:C_0805_2012Metric
- C19, C21: footprint (none) -> Capacitor_SMD:C_0603_1608Metric
- C2: footprint Capacitor_THT:CP_Radial_D8.0mm_P5.00mm -> Capacitor_SMD:C_0805_2012Metric
- C22, C9: footprint (none) -> Capacitor_SMD:C_0805_2012Metric
- D2, D8: footprint (none) -> LED_THT:LED_D5.0mm
Connections:
- net +3.3V: now also C5.1
- net +3V3B: now also C10.1, C4.1
- net GND: now also C11.1, C16.1, C17.1, C5.2, R1.2
- net GNDB: now also C10.2, C4.2
- net Piezzo_sens_1: now also C17.2, R1.1
- net at C21.2, C22.2, U4.2 (VCC)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: now also C11.2, C16.2

Commit message: 12/05/16:18
Parts:
- C1, C18, C7, C8: footprint Capacitor_SMD:C_0805_2012Metric -> Capacitor_SMD:C_1206_3216Metric
- C19, C21: footprint Capacitor_SMD:C_0603_1608Metric -> Capacitor_THT:C_Radial_D5.0mm_H11.0mm_P2.00mm
- C2: footprint Capacitor_SMD:C_0805_2012Metric -> Capacitor_THT:C_Radial_D5.0mm_H11.0mm_P2.00mm
- D1: footprint Diode_SMD:D_SMA -> Diode_SMD:D_SMC
- L1: footprint Inductor_THT:L_Radial_D10.0mm_P5.00mm_Fastron_07M -> Inductor_THT:L_Radial_D12.0mm_P5.00mm_Fastron_11P
Changed lines of the file:
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@@
 	(text "UART-USB"
 		(exclude_from_sim no)
-		(at 226.822 124.206 0)
+		(at 229.362 132.08 0)
 		(effects
 			(font
@@
 	(polyline
 		(pts
-			(xy 205.994 117.983) (xy 205.994 124.46)
+			(xy 205.74 124.46) (xy 205.74 124.46)
 		)
 		(stroke
@@
 	(polyline
 		(pts
-			(xy 205.994 12.7) (xy 205.994 117.983)
+			(xy 205.74 12.7) (xy 205.74 124.46)
 		)
 		(stroke
@@
 	(polyline
 		(pts
-			(xy 205.994 117.983) (xy 407.924 117.983)
+			(xy 205.74 124.46) (xy 407.67 124.46)
 		)
 		(stroke
@@
 			)
 		)
-		(property "Footprint" "Capacitor_SMD:C_0805_2012Metric"
+		(property "Footprint" "Capacitor_THT:C_Radial_D5.0mm_H11.0mm_P2.00mm"
 			(at 105.41 154.94 0)
 			(effects
@@
 			)
 		)
-		(property "Footprint" "Capacitor_SMD:C_0805_2012Metric"
+		(property "Footprint" "Capacitor_SMD:C_1206_3216Metric"
 			(at 26.67 154.94 0)
 			(effects
@@
 			)
 		)
-		(property "Footprint" "Inductor_THT:L_Radial_D10.0mm_P5.00mm_Fastron_07M"
+		(property "Footprint" "Inductor_THT:L_Radial_D12.0mm_P5.00mm_Fastron_11P"
 			(at 97.79 147.32 0)
 			(effects
@@
 			)
 		)
-		(property "Footprint" "Capacitor_SMD:C_0603_1608Metric"
+		(property "Footprint" "Capacitor_THT:C_Radial_D5.0mm_H11.0mm_P2.00mm"
 			(at 228.6 36.83 0)
 			(effects
@@
 			)
 		)
-		(property "Footprint" "Capacitor_SMD:C_0603_1608Metric"
+		(property "Footprint" "Capacitor_THT:C_Radial_D5.0mm_H11.0mm_P2.00mm"
 			(at 284.48 36.83 0)
 			(effects
@@
 			)
 		)
-		(property "Footprint" "Capacitor_SMD:C_0805_2012Metric"
+		(property "Footprint" "Capacitor_SMD:C_1206_3216Metric"
 			(at 40.64 154.94 0)
 			(effects
@@
 			)
 		)
-		(property "Footprint" "Diode_SMD:D_SMA"
+		(property "Footprint" "Diode_SMD:D_SMC"
 			(at 84.455 153.67 0)
 			(effects
@@
 			)
 		)
-		(property "Footprint" "Capacitor_SMD:C_0805_2012Metric"
+		(property "Footprint" "Capacitor_SMD:C_1206_3216Metric"
 			(at 151.4348 152.4 0)
 			(effects
@@
 			)
 		)
-		(property "Footprint" "Capacitor_SMD:C_0805_2012Metric"
+		(property "Footprint" "Capacitor_SMD:C_1206_3216Metric"
 			(at 176.8348 152.4 0)
 			(effects
