File: rs_485_proje.kicad_pcb (KiCad board)
At the start: 2 copper layers, 67.5 x 36 mm, 35 parts, among them J2 RJ45_LED, U1 AP2112K-3.3, U2 STM32G030F6Px, U3 SN65HVD1781, U5 TPS5420D, U7 PS8802-2

Commit message: 09/06/21:32
Parts:
- added C10: 100nF, Capacitor_SMD:C_0805_2012Metric, F.Cu at (245.3, 132.1)
- added C11: 100nF, Capacitor_SMD:C_0805_2012Metric, F.Cu at (249.7, 117.1)
- added C12: 100nF, Capacitor_SMD:C_0805_2012Metric, F.Cu at (249.7, 120.1)
- added C13: 100nF, Capacitor_SMD:C_0805_2012Metric, F.Cu at (249.7, 123.1)
- added C14: 100nF, Capacitor_SMD:C_0805_2012Metric, F.Cu at (249.7, 126.1)
- added C15: 100nf, Capacitor_SMD:C_0805_2012Metric, F.Cu at (249.7, 129.1)
- added C16: 100nF, Capacitor_SMD:C_0805_2012Metric, F.Cu at (249.7, 132.1)
- added C17: 4.7nf, Capacitor_SMD:C_0805_2012Metric, F.Cu at (254.2, 117.1)
- added C18: 4.7uf, Capacitor_SMD:C_1206_3216Metric, F.Cu at (238.1, 129.1)
- added C19: 10uf, Capacitor_THT:C_Radial_D5.0mm_H11.0mm_P2.00mm, F.Cu at (263.4, 123.4)
- added C20: 4.7nf, Capacitor_SMD:C_0805_2012Metric, F.Cu at (254.2, 120.1)
- added C21: 10uf, Capacitor_THT:C_Radial_D5.0mm_H11.0mm_P2.00mm, F.Cu at (263.4, 130.0)
- added C22: 10nf, Capacitor_SMD:C_0805_2012Metric, F.Cu at (254.2, 123.1)
- added C3: 100nF, Capacitor_SMD:C_0805_2012Metric, F.Cu at (245.3, 117.1)
- added C4: 100nF, Capacitor_SMD:C_0805_2012Metric, F.Cu at (245.3, 120.1)
- added C5: 100nF, Capacitor_SMD:C_0805_2012Metric, F.Cu at (245.3, 123.1)
- added C6: 100nF, Capacitor_SMD:C_0805_2012Metric, F.Cu at (245.3, 126.1)
- added C9: 10nf, Capacitor_SMD:C_0805_2012Metric, F.Cu at (245.3, 129.1)
- added D11: BZX84Cxx, Package_TO_SOT_SMD:SOT-23, F.Cu at (276.5, 112.3)
- added D14: BZX84Cxx, Package_TO_SOT_SMD:SOT-23, F.Cu at (276.5, 116.8)
- added D15: 1N5819, Diode_THT:D_DO-41_SOD81_P10.16mm_Horizontal, F.Cu at (244.9, 103.5)
- added D2: LED, LED_SMD:LED_0805_2012Metric_Pad1.15x1.40mm_HandSolder, F.Cu at (232.9, 129.0)
- added D3: 1N5819, Diode_THT:D_DO-41_SOD81_P10.16mm_Horizontal, F.Cu at (244.9, 82.3)
- added D4: 1N5819, Diode_THT:D_DO-41_SOD81_P10.16mm_Horizontal, F.Cu at (244.9, 86.5)
- added D5: 1N5819, Diode_THT:D_DO-41_SOD81_P10.16mm_Horizontal, F.Cu at (244.9, 90.8)
- added D6: SM712_SOT23, Package_TO_SOT_SMD:SOT-23, F.Cu at (276.5, 107.9)
- added D7: 1N5819, Diode_THT:D_DO-41_SOD81_P10.16mm_Horizontal, F.Cu at (244.9, 95.0)
- added D8: LED, LED_SMD:LED_0805_2012Metric_Pad1.15x1.40mm_HandSolder, F.Cu at (232.9, 132.0)
- added D9: 1N5819, Diode_THT:D_DO-41_SOD81_P10.16mm_Horizontal, F.Cu at (244.9, 99.3)
- added J1: xt60_female, Connector_AMASS:AMASS_XT60-F_1x02_P7.20mm_Vertical, F.Cu at (266.5, 85.3)
- added J10: Extra_pins, Connector_PinHeader_2.54mm:PinHeader_1x06_P2.54mm_Vertical, F.Cu at (258.7, 117.9)
- added J12: P_E_SENSOR_2, TerminalBlock_Phoenix:TerminalBlock_Phoenix_PT-1,5-2-3.5-H_1x02_P3.50mm_Horizontal, F.Cu at (254.9, 109.8)
- added J3: xt60_male, Connector_AMASS:AMASS_XT60-M_1x02_P7.20mm_Vertical, F.Cu at (266.5, 95.5)
- added J4: Led_conn, TerminalBlock_Phoenix:TerminalBlock_Phoenix_PT-1,5-3-3.5-H_1x03_P3.50mm_Horizontal, F.Cu at (233.3, 84.3)
- added J5: P_E_SENSOR_1, TerminalBlock_Phoenix:TerminalBlock_Phoenix_PT-1,5-2-3.5-H_1x02_P3.50mm_Horizontal, F.Cu at (245.8, 109.8)
- added J6: USB_B_Mini, Connector_USB:USB_Mini-B_Tensility_54-00023_Vertical_CircularHoles, F.Cu at (197.8, 139.0)
- added J7: H_E_sensor_1, TerminalBlock_Phoenix:TerminalBlock_Phoenix_PT-1,5-3-3.5-H_1x03_P3.50mm_Horizontal, F.Cu at (233.3, 94.2)
- added J8: H_E_sensor_2, TerminalBlock_Phoenix:TerminalBlock_Phoenix_PT-1,5-3-3.5-H_1x03_P3.50mm_Horizontal, F.Cu at (233.3, 104.1)
- added J9: Debug, Connector_PinHeader_2.54mm:PinHeader_1x04_P2.54mm_Vertical, F.Cu at (270.0, 122.4)
- added R1: 1M, Resistor_SMD:R_0805_2012Metric, F.Cu at (259.2, 81.6)
- added R15: 330R, Resistor_SMD:R_0805_2012Metric, F.Cu at (259.2, 84.6)
- added R16: 330R, Resistor_SMD:R_0805_2012Metric, F.Cu at (259.2, 87.5)
- added R18: 1M, Resistor_SMD:R_0805_2012Metric, F.Cu at (259.2, 90.5)
- added R19: 120R, Resistor_SMD:R_0805_2012Metric, F.Cu at (259.2, 93.4)
- added R20: 330R, Resistor_SMD:R_0805_2012Metric, F.Cu at (259.2, 96.4)
- added R21: 10K, Resistor_SMD:R_0805_2012Metric, F.Cu at (259.2, 99.3)
- added U10: FT232RL, Package_SO:SSOP-28_5.3x10.2mm_P0.65mm, F.Cu at (235.7, 115.8)
- added U11: USBLC6-2SC6, Package_TO_SOT_SMD:SOT-23-6, F.Cu at (274.9, 122.5)
- added U4: ADM2587E, Package_SO:SOIC-20W_7.5x12.8mm_P1.27mm, F.Cu at (267.6, 113.0)
- C1: value 10uf -> 4.7uf; footprint Capacitor_THT:C_Radial_D5.0mm_H11.0mm_P2.00mm -> Capacitor_SMD:C_1206_3216Metric
- C2: footprint Capacitor_THT:CP_Radial_D8.0mm_P5.00mm -> Capacitor_THT:C_Radial_D5.0mm_H11.0mm_P2.00mm
- C7: footprint Capacitor_SMD:C_0805_2012Metric -> Capacitor_SMD:C_1206_3216Metric_Pad1.33x1.80mm_HandSolder
- C8: footprint Capacitor_SMD:C_0805_2012Metric -> Capacitor_SMD:C_1206_3216Metric
- D1: footprint Diode_SMD:D_SMA -> Diode_SMD:D_SMC
- J2: footprint Connector_RJ:RJ45_Wuerth_7499010001A_Horizontal -> Connector_RJ:RJ45_Connfly_DS1128-09-S8xx-S_Horizontal
- L1: footprint Inductor_THT:L_Radial_D10.0mm_P5.00mm_Fastron_07M -> Inductor_THT:L_Radial_D12.0mm_P5.00mm_Fastron_11P
- U7: value PS8802-2 -> TLP2161
Connections:
- C2 pad 1: +5V -> Net-(C2-Pad1)
- C7 pad 2: +5V -> Net-(U1-EN)
- J2 pad 1: unconnected-(J2-Pad1) -> /RS485_A(-)
- J2 pad 10: (no net) -> Net-(J2-Pad10)
- J2 pad 11: (no net) -> GND
- J2 pad 12: (no net) -> Net-(J2-Pad12)
- J2 pad 2: unconnected-(J2-Pad2) -> /RS485_B(+)
- J2 pad 3: unconnected-(J2-Pad3) -> GNDB
- J2 pad 7: unconnected-(J2-Pad7) -> +24V
- J2 pad 8: unconnected-(J2-Pad8) -> GND
- J2 pad 9: (no net) -> GND
- L1 pad 2: +5V -> Net-(C2-Pad1)
- R11 pad 2: /Digital_sens_1 -> Net-(J7-Pin_2)
- R12 pad 1: +5V -> Net-(R12-Pad1)
- R12 pad 2: /Digital_sens_2 -> Net-(J8-Pin_2)
- R13 pad 1: /SENS_3 -> /Digital_sens_1
- R14 pad 1: /SENS_4 -> /Digital_sens_2
- R4 pad 1: +5V -> Net-(R4-Pad1)
- U1 pad 1: +5V -> Net-(U1-EN)
- U1 pad 3: +5V -> Net-(U1-EN)
- U2 pad 13: /Extra_4 -> /PA_6
- U2 pad 14: /Extra_3 -> /PA_7
- U2 pad 15: /Extra_2 -> /RS_485_D_EN
- U2 pad 16: /Extra_1 -> /RS_485_R_EN
- U2 pad 17: /RS_485_D_EN -> /LED_Driver
- U2 pad 18: /RS_485_R_EN -> /SWDIO
- U2 pad 19: /LED_Driver -> /SWCLK
- U2 pad 3: /RS_485_RX_LED -> /RS_485_TX_LED
- U7 pad 1: /Digital_sens_1 -> Net-(J7-Pin_2)
- U7 pad 3: /Digital_sens_2 -> GND
- U7 pad 4: GND -> Net-(J8-Pin_2)
- U7 pad 6: /SENS_4 -> /Digital_sens_2
- U7 pad 7: /SENS_3 -> /Digital_sens_1

Commit message: 10/06/13:37
Parts:
- added C19: 10uf, Capacitor_SMD:C_0805_2012Metric_Pad1.18x1.45mm_HandSolder, F.Cu at (252.0, 79.0)
- added C23: 10uf, Capacitor_SMD:C_0805_2012Metric_Pad1.18x1.45mm_HandSolder, F.Cu at (252.5, 85.0)
- C1, C18, C8: footprint Capacitor_SMD:C_1206_3216Metric -> Capacitor_SMD:C_0805_2012Metric_Pad1.18x1.45mm_HandSolder
- C10, C11, C12, C13, C14, C15, C16, C17, C20, C22, C3, C4, C5, C6, C9: footprint Capacitor_SMD:C_0805_2012Metric -> Capacitor_SMD:C_0805_2012Metric_Pad1.18x1.45mm_HandSolder
- C7: footprint Capacitor_SMD:C_1206_3216Metric_Pad1.33x1.80mm_HandSolder -> Capacitor_SMD:C_0805_2012Metric_Pad1.18x1.45mm_HandSolder
- D15, D3, D4, D5, D7, D9: footprint Diode_THT:D_DO-41_SOD81_P10.16mm_Horizontal -> Diode_SMD:D_SOD-123
- R1, R10, R11, R12, R13, R14, R15, R16, R18, R19, R20, R21, R4, R5, R7, R9: footprint Resistor_SMD:R_0805_2012Metric -> Resistor_SMD:R_0805_2012Metric_Pad1.20x1.40mm_HandSolder
- moved D1 10.1 mm to (203.0, 121.5)
